File: PCB/PCB.kicad_sch (KiCad schematic)
At the start: 1 part, among them U1 STM32F072CBTx

Commit message: Update PCB
Parts:
- removed U1: STM32F072CBTx, Package_QFP:LQFP-48_7x7mm_P0.5mm, symbol MCU_ST_STM32F0:STM32F072CBTx
- added F1: Fuse, symbol Device:Fuse
- added J1: USB_C_Receptacle_USB2.0_16P, symbol Connector:USB_C_Receptacle_USB2.0_16P
- added J2, J3: Conn_01x20, symbol Connector_Generic:Conn_01x20
- added J4: SSD1306, symbol Connector_Generic:Conn_01x04
- added R2, R3: 5k1, symbol Device:R
- added SW1, SW2: SW_Push, symbol Switch:SW_Push
- added U2: USBLC6-2SC6, Package_TO_SOT_SMD:SOT-23-6, symbol Power_Protection:USBLC6-2SC6
Connections:
- new net: J1.B5 (CC2), R3.1
- new net: J1.A6 (D+), J1.B6 (D+), U2.1 (I/O1)
- new net: J1.A7 (D-), J1.B7 (D-), U2.3 (I/O2)
- new net: J1.A5 (CC1), R2.1
- new net +3.3V: J3.20 (Pin_20), J4.2 (Pin_2)
- new net +5V: F1.2, J3.18 (Pin_18), U2.5 (VBUS)
- new net D+: J3.9 (Pin_9), U2.6 (I/O1)
- new net D-: J3.8 (Pin_8), U2.4 (I/O2)
- new net GND: J1.A1 (GND), J1.A12 (GND), J1.B1 (GND), J1.B12 (GND), J1.S1 (SHIELD), J2.19 (Pin_19), J2.20 (Pin_20), J3.19 (Pin_19), J4.1 (Pin_1), R2.2, R3.2, SW1.2, SW2.2, U2.2 (GND)
- new net S1: J2.11 (Pin_11), SW1.1
- new net S2: J2.12 (Pin_12), SW2.1
- new net SSD1306_SCL: J3.14 (Pin_14), J4.3 (Pin_3)
- new net SSD1306_SDA: J3.15 (Pin_15), J4.4 (Pin_4)
- new net VBUS: F1.1, J1.A4 (VBUS), J1.A9 (VBUS), J1.B4 (VBUS), J1.B9 (VBUS)
- no-connect marks 0 -> 2
Other:
- note added: "Decoupling Capacitors"
- note added: "Screen"
- note added: "Switches"
